File: InputSwitch.kicad_sch (KiCad schematic)
At the start: 10 parts, among them SW10 SW_B, SW11 SW_C, SW12 SW_D, SW13 SW_ENTER, SW8 RotaryEncoder, SW9 SW_A, U5 74HC14

Commit message: InputSwitchのスイッチ名称の変更が必要
Other:
- company: (none) -> LLC. YS-Lab.
- title: (none) -> InputSwitch Part
Changed lines of the file:
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@@
 (kicad_sch (version 20230121) (generator eeschema)
   (paper "A4")
+  (title_block
+    (title "InputSwitch Part")
+    (date "2024-02-16")
+    (rev "1.00")
+    (company "LLC. YS-Lab.")
+    (comment 1 "スイッチの名称を反映させる")
+  )
   (junction (at 163.83 95.25) (diameter 0) (color 0 0 0 0)
   )

Commit message: PCB配置作業中
Parts:
- C401: renamed from C6; footprint (none) -> Capacitor_THT:C_Disc_D3.0mm_W2.0mm_P2.50mm
- C402: renamed from C8; footprint (none) -> Capacitor_THT:C_Disc_D3.0mm_W2.0mm_P2.50mm
- C403: renamed from C7; footprint (none) -> Capacitor_THT:C_Disc_D3.0mm_W2.0mm_P2.50mm
- SW402: renamed from SW9; value SW_A -> SW_UP
- SW403: renamed from SW10; value SW_B -> SW_DOWN
- SW404: renamed from SW11; value SW_C -> SW_LEFT
- SW405: renamed from SW12; value SW_D -> SW_RIGHT
- U401: renamed from U5; footprint (none) -> Package_DIP:DIP-14_W7.62mm_LongPads
- renumbered SW8 to SW401, SW13 to SW406, U5 to U401
Connections:
- net SW_A renamed SW_UP
- net SW_B renamed SW_DOWN
- net SW_C renamed SW_LEFT
- net SW_D renamed SW_RIGHT
Changed lines of the file:
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@@
     (effects (font (size 1.27 1.27)) (justify left))
   )
-  (hierarchical_label "SW_D" (shape input) (at 196.85 140.97 0) (fields_autoplaced)
-    (effects (font (size 1.27 1.27)) (justify left))
-  )
-  (hierarchical_label "SW_A" (shape input) (at 196.85 106.68 0) (fields_autoplaced)
+  (hierarchical_label "SW_RIGHT" (shape input) (at 196.85 140.97 0) (fields_autoplaced)
+    (effects (font (size 1.27 1.27)) (justify left))
+  )
+  (hierarchical_label "SW_UP" (shape input) (at 196.85 106.68 0) (fields_autoplaced)
     (effects (font (size 1.27 1.27)) (justify left))
   )
@@
     (effects (font (size 1.27 1.27)) (justify left))
   )
-  (hierarchical_label "SW_C" (shape input) (at 196.85 129.54 0) (fields_autoplaced)
-    (effects (font (size 1.27 1.27)) (justify left))
-  )
-  (hierarchical_label "SW_B" (shape input) (at 196.85 118.11 0) (fields_autoplaced)
+  (hierarchical_label "SW_LEFT" (shape input) (at 196.85 129.54 0) (fields_autoplaced)
+    (effects (font (size 1.27 1.27)) (justify left))
+  )
+  (hierarchical_label "SW_DOWN" (shape input) (at 196.85 118.11 0) (fields_autoplaced)
     (effects (font (size 1.27 1.27)) (justify left))
   )
@@
   (symbol (lib_id "Device:C_Small") (at 148.59 90.17 0) (unit 1)
     (in_bom yes) (on_board yes) (dnp no) (fields_autoplaced)
-    (property "Reference" "C8" (at 150.9141 88.9642 0)
+    (property "Reference" "C402" (at 150.9141 88.9642 0)
       (effects (font (size 1.27 1.27)) (justify left))
     )
@@
       (effects (font (size 1.27 1.27)) (justify left))
     )
-    (property "Footprint" "" (at 148.59 90.17 0)
+    (property "Footprint" "Capacitor_THT:C_Disc_D3.0mm_W2.0mm_P2.50mm" (at 148.59 90.17 0)
       (effects (font (size 1.27 1.27)) hide)
     )
@@
       (project "M304B"
         (path "/922fb1f0-ef32-4fe1-b104-d5a058d25ebb/808aea72-aba1-451d-966a-43c6afccf196"
-          (reference "C8") (unit 1)
+          (reference "C402") (unit 1)
         )
       )
@@
   (symbol (lib_id "Device:C_Small") (at 163.83 90.17 0) (unit 1)
     (in_bom yes) (on_board yes) (dnp no) (fields_autoplaced)
-    (property "Reference" "C7" (at 166.1541 88.9642 0)
+    (property "Reference" "C403" (at 166.1541 88.9642 0)
       (effects (font (size 1.27 1.27)) (justify left))
     )
@@
       (effects (font (size 1.27 1.27)) (justify left))
     )
-    (property "Footprint" "" (at 163.83 90.17 0)
+    (property "Footprint" "Capacitor_THT:C_Disc_D3.0mm_W2.0mm_P2.50mm" (at 163.83 90.17 0)
       (effects (font (size 1.27 1.27)) hide)
     )
@@
       (project "M304B"
         (path "/922fb1f0-ef32-4fe1-b104-d5a058d25ebb/808aea72-aba1-451d-966a-43c6afccf196"
-          (reference "C7") (unit 1)
+          (reference "C403") (unit 1)
         )
       )
@@
   (symbol (lib_id "Switch:SW_SPST") (at 180.34 118.11 0) (unit 1)
     (in_bom yes) (on_board yes) (dnp no)
-    (property "Reference" "SW10" (at 176.53 116.84 0)
-      (effects (font (size 1 1)))
-    )
-    (property "Value" "SW_B" (at 185.42 116.84 0)
+    (property "Reference" "SW403" (at 176.53 116.84 0)
+      (effects (font (size 1 1)))
+    )
+    (property "Value" "SW_DOWN" (at 186.69 116.84 0)
       (effects (font (size 1 1)))
     )
@@
       (project "M304B"
         (path "/922fb1f0-ef32-4fe1-b104-d5a058d25ebb/808aea72-aba1-451d-966a-43c6afccf196"
-          (reference "SW10") (unit 1)
+          (reference "SW403") (unit 1)
         )
       )
@@
   (symbol (lib_id "Switch:SW_SPST") (at 180.34 152.4 0) (unit 1)
     (in_bom yes) (on_board yes) (dnp no)
-    (property "Reference" "SW13" (at 176.53 151.13 0)
-      (effects (font (size 1 1)))
-    )
-    (property "Value" "SW_ENTER" (at 185.42 151.13 0)
+    (property "Reference" "SW406" (at 176.53 151.13 0)
+      (effects (font (size 1 1)))
+    )
+    (property "Value" "SW_ENTER" (at 186.69 151.13 0)
       (effects (font (size 1 1)))
     )
@@
       (project "M304B"
         (path "/922fb1f0-ef32-4fe1-b104-d5a058d25ebb/808aea72-aba1-451d-966a-43c6afccf196"
-          (reference "SW13") (unit 1)
+          (reference "SW406") (unit 1)
         )
       )
@@
   (symbol (lib_id "74xx:74HC14") (at 177.8 71.12 0) (unit 2)
     (in_bom yes) (on_board yes) (dnp no) (fields_autoplaced)
-    (property "Reference" "U5" (at 177.8 63.1657 0)
+    (property "Reference" "U401" (at 177.8 63.1657 0)
       (effects (font (size 1.27 1.27)))
     )
@@
       (project "M304B"
         (path "/922fb1f0-ef32-4fe1-b104-d5a058d25ebb/808aea72-aba1-451d-966a-43c6afccf196"
-          (reference "U5") (unit 2)
+          (reference "U401") (unit 2)
         )
       )
@@
   (symbol (lib_id "Device:RotaryEncoder") (at 151.13 40.64 90) (unit 1)
     (in_bom yes) (on_board yes) (dnp no) (fields_autoplaced)
-    (property "Reference" "SW8" (at 156.972 39.4279 90)
+    (property "Reference" "SW401" (at 156.972 39.4279 90)
       (effects (font (size 1.27 1.27)) (justify right))
     )
@@
       (project "M304B"
         (path "/922fb1f0-ef32-4fe1-b104-d5a058d25ebb/808aea72-aba1-451d-966a-43c6afccf196"
-          (reference "SW8") (unit 1)
+          (reference "SW401") (unit 1)
         )
       )
@@
   (symbol (lib_id "Switch:SW_SPST") (at 180.34 140.97 0) (unit 1)
     (in_bom yes) (on_board yes) (dnp no)
-    (property "Reference" "SW12" (at 176.53 139.7 0)
-      (effects (font (size 1 1)))
-    )
-    (property "Value" "SW_D" (at 185.42 139.7 0)
+    (property "Reference" "SW405" (at 176.53 139.7 0)
+      (effects (font (size 1 1)))
+    )
+    (property "Value" "SW_RIGHT" (at 186.69 139.7 0)
       (effects (font (size 1 1)))
     )
@@
       (project "M304B"
         (path "/922fb1f0-ef32-4fe1-b104-d5a058d25ebb/808aea72-aba1-451d-966a-43c6afccf196"
-          (reference "SW12") (unit 1)
+          (reference "SW405") (unit 1)
         )
       )
@@
   (symbol (lib_id "74xx:74HC14") (at 129.54 50.8 0) (unit 7)
     (in_bom yes) (on_board yes) (dnp no) (fields_autoplaced)
-    (property "Reference" "U5" (at 135.382 49.5879 0)
+    (property "Reference" "U401" (at 135.382 49.5879 0)
       (effects (font (size 1.27 1.27)) (justify left))
     )
@@
       (effects (font (size 1.27 1.27)) (justify left))
     )
-    (property "Footprint" "" (at 129.54 50.8 0)
+    (property "Footprint" "Package_DIP:DIP-14_W7.62mm_LongPads" (at 129.54 50.8 0)
       (effects (font (size 1.27 1.27)) hide)
     )
@@
       (project "M304B"
         (path "/922fb1f0-ef32-4fe1-b104-d5a058d25ebb/808aea72-aba1-451d-966a-43c6afccf196"
-          (reference "U5") (unit 7)
+          (reference "U401") (unit 7)
         )
       )
@@
   (symbol (lib_id "Switch:SW_SPST") (at 180.34 106.68 0) (unit 1)
     (in_bom yes) (on_board yes) (dnp no)
-    (property "Reference" "SW9" (at 176.53 105.41 0)
-      (effects (font (size 1 1)))
-    )
-    (property "Value" "SW_A" (at 185.42 105.41 0)
+    (property "Reference" "SW402" (at 176.53 105.41 0)
+      (effects (font (size 1 1)))
+    )
+    (property "Value" "SW_UP" (at 185.42 105.41 0)
       (effects (font (size 1 1)))
     )
@@
       (project "M304B"
         (path "/922fb1f0-ef32-4fe1-b104-d5a058d25ebb/808aea72-aba1-451d-966a-43c6afccf196"
-          (reference "SW9") (unit 1)
+          (reference "SW402") (unit 1)
         )
       )
@@
   (symbol (lib_id "Device:C_Small") (at 115.57 50.8 0) (unit 1)
     (in_bom yes) (on_board yes) (dnp no) (fields_autoplaced)
-    (property "Reference" "C6" (at 117.8941 49.5942 0)
+    (property "Reference" "C401" (at 117.8941 49.5942 0)
       (effects (font (size 1.27 1.27)) (justify left))
     )
@@
       (effects (font (size 1.27 1.27)) (justify left))
     )
-    (property "Footprint" "" (at 115.57 50.8 0)
+    (property "Footprint" "Capacitor_THT:C_Disc_D3.0mm_W2.0mm_P2.50mm" (at 115.57 50.8 0)
       (effects (font (size 1.27 1.27)) hide)
     )
@@
       (project "M304B"
         (path "/922fb1f0-ef32-4fe1-b104-d5a058d25ebb/808aea72-aba1-451d-966a-43c6afccf196"
-          (reference "C6") (unit 1)
+          (reference "C401") (unit 1)
         )
       )
@@
   (symbol (lib_id "Switch:SW_SPST") (at 180.34 129.54 0) (unit 1)
     (in_bom yes) (on_board yes) (dnp no)
-    (property "Reference" "SW11" (at 176.53 128.27 0)
-      (effects (font (size 1 1)))
-    )
-    (property "Value" "SW_C" (at 185.42 128.27 0)
+    (property "Reference" "SW404" (at 176.53 128.27 0)
+      (effects (font (size 1 1)))
+    )
+    (property "Value" "SW_LEFT" (at 186.69 128.27 0)
       (effects (font (size 1 1)))
     )
@@
       (project "M304B"
         (path "/922fb1f0-ef32-4fe1-b104-d5a058d25ebb/808aea72-aba1-451d-966a-43c6afccf196"
-          (reference "SW11") (unit 1)
+          (reference "SW404") (unit 1)
         )
       )
@@
   (symbol (lib_id "74xx:74HC14") (at 177.8 85.09 0) (unit 1)
     (in_bom yes) (on_board yes) (dnp no) (fields_autoplaced)
-    (property "Reference" "U5" (at 177.8 77.1357 0)
+    (property "Reference" "U401" (at 177.8 77.1357 0)
       (effects (font (size 1.27 1.27)))
     )
@@
       (project "M304B"
         (path "/922fb1f0-ef32-4fe1-b104-d5a058d25ebb/808aea72-aba1-451d-966a-43c6afccf196"
-          (reference "U5") (unit 1)
-        )
-      )
+          (reference "U401") (unit 1)
+        )
+      )

Commit message: 途中
Parts:
- removed U401: 74HC14, Package_DIP:DIP-14_W7.62mm_LongPads, symbol 74xx:74HC14
- added C404, C405, C406, C407, C408: 0.1uF, Capacitor_THT:C_Disc_D3.0mm_W2.0mm_P2.50mm, symbol Device:C_Small
- added R401, R402, R403, R404, R405, R406, R407, R408, R409, R410, R411, R412, R413, R414: 10k, symbol Device:R_US
Connections:
- net +5V: now also R401.1, R402.1, R410.2, R411.2, R412.2, R413.2, R414.2
- net GND: now also C404.2, C405.2, C406.2, C407.2, C408.2
- net RE_A: now also C402.1, R403.2
- net RE_B: now also C403.1, R404.2
- net SW_DOWN: now also C405.1, R406.2; no longer SW403.2 (B)
- net SW_ENTER: now also C408.1, R409.2; no longer SW406.2 (B)
- net SW_LEFT: now also C406.1, R407.2; no longer SW404.2 (B)
- net SW_RIGHT: now also C407.1, R408.2; no longer SW405.2 (B)
- net SW_UP: now also C404.1, R405.2; no longer SW402.2 (B)
- net at SW401.A: now also R401.2, R403.1; no longer C402.1
- net at SW401.B: now also R402.2, R404.1; no longer C403.1
- new net: R408.1, R413.1, SW405.2 (B)
- new net: R407.1, R412.1, SW404.2 (B)
- new net: R406.1, R411.1, SW403.2 (B)
- new net: R409.1, R414.1, SW406.2 (B)
- new net: R405.1, R410.1, SW402.2 (B)
Other:
- moved on the sheet: C402, C403, SW402, SW403, SW404, SW405, SW406
