File: M304B.kicad_sch (KiCad schematic)
At the start: 56 parts, among them J1 LCD 2004, J2 Relay OUT, J5 POWER IN, P1 Digital, P10 CONN_01X01, P11 CONN_01X01, P12 CONN_01X01, P13 CONN_01X01, P2 Power, P3 Analog, P4 Analog, P5 PWM, P6 PWM, P7 Communication, P8 CONN_01X01, P9 CONN_01X01, SW1 RESET, SW2 SW_A, SW3 SW_B, SW4 SW_C, SW5 SW_D, SW6 SW_ENTER, SW7 SAFEMODE, SW8 RotaryEncoder, U2 24LC256, U3 W5500, U4 LM1117-3.3, U5 74HC14

Commit message: もう少し
Parts:
- removed JD49: Conn_01x01, Connector_Pin:Pin_D0.9mm_L10.0mm_W2.4mm_FlatFork, symbol Connector_Generic:Conn_01x01
- removed SW2: SW_A, HOLLY:TVDT18-050, symbol Switch:SW_SPST
- removed SW3: SW_B, HOLLY:TVDT18-050, symbol Switch:SW_SPST
- removed SW4: SW_C, HOLLY:TVDT18-050, symbol Switch:SW_SPST
- removed SW5: SW_D, HOLLY:TVDT18-050, symbol Switch:SW_SPST
- removed SW6: SW_ENTER, HOLLY:TVDT18-050, symbol Switch:SW_SPST
- removed SW8: RotaryEncoder, Rotary_Encoder:RotaryEncoder_Alps_EC12E_Vertical_H20mm, symbol Device:RotaryEncoder
- removed U5: 74HC14, Package_DIP:DIP-14_W7.62mm_LongPads, symbol 74xx:74HC14
Connections:
- net 49: no longer P1.8 (Pin_8)
- net RE_A: now reaches P7.5 (Pin_5)
- net RE_B: now reaches P7.6 (Pin_6)
- net 32 renamed SW_ENTER
- net 34 renamed SW_B
- net 36 renamed SW_D
- no-connect marks 37 -> 35
Other:
- added sheet InputSwitch (InputSwitch.kicad_sch)
- company: AMPSD Kyushu Univ. -> AMPSD Kyushu Univ. YS-Lab
- title: M304 UECS Controller shield for Arduino MEGA SMANOU2022 -> M304B UECS Controller shield for Arduino MEGA BABY SIZE
- moved on the sheet: JP31, JP32, JP51, JP52, JP53

Commit message: 細かい整形
Connections:
- net +5V: no longer C2.2, C4.2, R2.1, R3.1, U2.8 (VCC), U4.3 (VI)
- net 10(**): now also P5.8 (Pin_8)
- net 11(**): now also P5.7 (Pin_7)
- net 12(**): now also P5.6 (Pin_6)
- net 13(**): now also P5.5 (Pin_5)
- net 14(Tx3): now also P7.1 (Pin_1)
- net 15(Rx3): now also P7.2 (Pin_2)
- net 2(**): now also P6.6 (Pin_6)
- net 4(**): now also P6.4 (Pin_4)
- net 49: now also P1.8 (Pin_8)
- net 5(**): now also P6.3 (Pin_3)
- net 6(**): now also P6.2 (Pin_2)
- net A10: now also P4.3 (Pin_3)
- net A11: now also P4.4 (Pin_4)
- net A12: now also P4.5 (Pin_5)
- net A13: now also P4.6 (Pin_6)
- net A14: now also P4.7 (Pin_7)
- net A15: now also P4.8 (Pin_8)
- net A2: now also P3.3 (Pin_3)
- net A3: now also P3.4 (Pin_4)
- net A4: now also P3.5 (Pin_5)
- net A5: now also P3.6 (Pin_6)
- net A6: now also P3.7 (Pin_7)
- net A7: now also P3.8 (Pin_8)
- new net: C4.2, U4.3 (VI)
- new net VCC: C2.2, R2.1, R3.1, U2.8 (VCC)
- no-connect marks 35 -> 39
Other:
- note added: "18(Tx1)"
- note added: "19(Rx1)"
- note added: "20"
- note added: "21"
- note added: "32"
- note added: "34"
- note added: "36"

Commit message: PCB配置作業中
Parts:
- P108: renamed from P8; now left out of the parts list
- P109: renamed from P9; now left out of the parts list
- P110: renamed from P10; now left out of the parts list
- P111: renamed from P11; now left out of the parts list
- P112: renamed from P12; now left out of the parts list
- P113: renamed from P13; now left out of the parts list
- renumbered C4 to C101, C3 to C102, C5 to C103, C2 to C104, D5 to D101, J5 to J101, J2 to J102, J1 to J103, JA0 to JA101, JA1 to JA102, JA8 to JA103, JA9 to JA104, JC1 to JC101, JC2 to JC102, JD30 to JD101, JD48 to JD102, JD9 to JD103, JD8 to JD104, JD7 to JD105, JP31 to JP101, JP32 to JP102, JP51 to JP103, JP52 to JP104, JP53 to JP105, JX2 to JX101, P2 to P101, P3 to P102, P4 to P103, P1 to P104, P5 to P105, P6 to P106, P7 to P107, R1 to R101, R2 to R102, R3 to R103, R7 to R104, RV1 to RV101, SW1 to SW101, SW7 to SW102, U4 to U101, U2 to U102, U3 to U103
Connections:
- net 22 renamed INPUT1
- net 24 renamed INPUT3
- net 26 renamed INPUT5
- net 28 renamed INPUT7
- net SW_B renamed SW_DOWN
- net SW_D renamed SW_RIGHT
Other:
- sheet InputSwitch ports: added SW_DOWN, SW_LEFT, SW_RIGHT, SW_UP; removed SW_A, SW_B, SW_C, SW_D
- note added: "22"
- note added: "24"
- note added: "26"
- note added: "28"
- moved on the sheet: JD101, JD102
