File: RTC.kicad_sch (KiCad schematic)
At the start: 5 parts, among them U1 DS1307+, Y1 32.768kHz

Commit message: もう少し
Parts:
- added D1: 1N4148, Diode_THT:D_DO-35_SOD27_P7.62mm_Horizontal, symbol Diode:1N4148
- added JP1, JP2: CR or LIR, symbol Jumper:Jumper_3_Open
- added R4: 200, symbol Device:R_US
- added R5: 1.8M, symbol Device:R_US
- added R6: 1.8k, symbol Device:R_US
- added R8: 680k, symbol Device:R_US
- added R9: 470k, symbol Device:R_US
Connections:
- net +5V: now also R4.2, R8.1
- net GND: now also R5.2, R6.2
- net at U1.2 (X2), Y1.2: now also R8.2
- net at BT1.1 (+): now also JP1.2 (C); no longer U1.3 (VBAT)
- new net: D1.1 (K), JP1.1 (A), R9.1
- new net: JP2.1 (A), R5.1, R9.2
- new net: JP1.3 (B), JP2.3 (B)
- new net: D1.2 (A), R4.1, R6.1
- new net: JP2.2 (C), U1.3 (VBAT)
Other:
- moved on the sheet: BT1, SQW1

Commit message: 細かい整形
Parts:
- JP1, JP2: value CR or LIR -> LIR or CR
Connections:
- net VBAT: now reaches JP2.2 (C), U1.3 (VBAT)
Changed lines of the file:
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@@
     (effects (font (size 1.27 1.27)) (justify left bottom))
   )
+  (label "VBAT" (at 109.22 74.93 0) (fields_autoplaced)
+    (effects (font (size 1.27 1.27)) (justify left bottom))
+  )
   (hierarchical_label "SDA" (shape bidirectional) (at 172.72 86.36 0) (fields_autoplaced)
     (effects (font (size 1.27 1.27)) (justify left))
   )
-  (hierarchical_label "+5V" (shape input) (at 135.89 57.15 90) (fields_autoplaced)
+  (hierarchical_label "+5V" (shape output) (at 135.89 57.15 90) (fields_autoplaced)
     (effects (font (size 1.27 1.27)) (justify left))
   )
@@
   (symbol (lib_id "Jumper:Jumper_3_Open") (at 71.12 82.55 0) (unit 1)
     (in_bom yes) (on_board yes) (dnp no) (fields_autoplaced)
-    (property "Reference" "JP1" (at 71.12 77.0335 0)
-      (effects (font (size 1.27 1.27)))
-    )
-    (property "Value" "CR or LIR" (at 71.12 79.4577 0)
+    (property "Reference" "JP1" (at 71.12 76.2 0)
+      (effects (font (size 1.27 1.27)))
+    )
+    (property "Value" "LIR or CR" (at 71.12 78.74 0)
       (effects (font (size 1.27 1.27)))
     )
@@
     )
   )
-  (symbol (lib_id "Jumper:Jumper_3_Open") (at 107.95 68.58 0) (unit 1)
-    (in_bom yes) (on_board yes) (dnp no) (fields_autoplaced)
-    (property "Reference" "JP2" (at 107.95 63.0635 0)
-      (effects (font (size 1.27 1.27)))
-    )
-    (property "Value" "CR or LIR" (at 107.95 65.4877 0)
+  (symbol (lib_name "Jumper_3_Open_1") (lib_id "Jumper:Jumper_3_Open") (at 107.95 68.58 0) (unit 1)
+    (in_bom yes) (on_board yes) (dnp no) (fields_autoplaced)
+    (property "Reference" "JP2" (at 107.95 62.23 0)
+      (effects (font (size 1.27 1.27)))
+    )
+    (property "Value" "LIR or CR" (at 107.95 64.77 0)
       (effects (font (size 1.27 1.27)))
     )
@@
       (project "M304B"
         (path "/922fb1f0-ef32-4fe1-b104-d5a058d25ebb/1e2511a2-7248-4cea-afb1-80995e2b8f5b"
+          (reference "JP2") (unit 1)
+        )
+        (path "/922fb1f0-ef32-4fe1-b104-d5a058d25ebb"
           (reference "JP2") (unit 1)
         )
@@
       (effects (font (size 1.27 1.27)) (justify left))
     )
-    (property "Footprint" "Akizuki:CH74-2032LF" (at 71.12 92.456 90)
-      (effects (font (size 1.27 1.27)) hide)
-    )
+    (property "Footprint" "Akizuki:CH74-2032LF" (at 72.39 97.79 0)
+      (effects (font (size 1.27 1.27)) hide)
+    )

Commit message: InputSwitchのスイッチ名称の変更が必要
Other:
- company: HOLLY&Co.,Ltd. -> LLC. YS-Lab
Changed lines of the file:
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@@
   (title_block
     (title "RTC回路")
-    (date "2022-08-02")
-    (rev "1.00")
-    (company "HOLLY&Co.,Ltd.")
+    (date "2024-02-16")
+    (rev "2.00")
+    (company "LLC. YS-Lab")
+    (comment 1 "LIRを使用するときはJP1,2を1-2をショート CRを使用するときは2-3をショート")
   )
   (junction (at 166.37 96.52) (diameter 0) (color 0 0 0 0)
@@
           (reference "JP2") (unit 1)
         )
-        (path "/922fb1f0-ef32-4fe1-b104-d5a058d25ebb"
-          (reference "JP2") (unit 1)
-        )

Commit message: PCB配置作業中
Parts:
- JP301: renamed from JP1; footprint (none) -> Connector_PinHeader_2.54mm:PinHeader_1x03_P2.54mm_Vertical
- JP302: renamed from JP2; footprint (none) -> Connector_PinHeader_2.54mm:PinHeader_1x03_P2.54mm_Vertical
- R301: renamed from R6; footprint (none) -> Resistor_THT:R_Axial_DIN0207_L6.3mm_D2.5mm_P7.62mm_Horizontal
- R302: renamed from R4; footprint (none) -> Resistor_THT:R_Axial_DIN0207_L6.3mm_D2.5mm_P7.62mm_Horizontal
- R303: renamed from R9; footprint (none) -> Resistor_THT:R_Axial_DIN0207_L6.3mm_D2.5mm_P7.62mm_Horizontal
- R304: renamed from R5; footprint (none) -> Resistor_THT:R_Axial_DIN0207_L6.3mm_D2.5mm_P7.62mm_Horizontal
- R305: renamed from R8; footprint (none) -> Resistor_THT:R_Axial_DIN0207_L6.3mm_D2.5mm_P7.62mm_Horizontal
- renumbered BT1 to BT301, C1 to C301, D1 to D301, SQW1 to SQW301, U1 to U301, Y1 to Y301
Changed lines of the file:
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@@
   (symbol (lib_id "Device:R_US") (at 88.9 74.93 90) (unit 1)
     (in_bom yes) (on_board yes) (dnp no) (fields_autoplaced)
-    (property "Reference" "R9" (at 88.9 69.8967 90)
+    (property "Reference" "R303" (at 88.9 69.8967 90)
       (effects (font (size 1.27 1.27)))
     )
@@
       (effects (font (size 1.27 1.27)))
     )
-    (property "Footprint" "" (at 89.154 73.914 90)
+    (property "Footprint" "Resistor_THT:R_Axial_DIN0207_L6.3mm_D2.5mm_P7.62mm_Horizontal" (at 89.154 73.914 90)
       (effects (font (size 1.27 1.27)) hide)
     )
@@
       (project "M304B"
         (path "/922fb1f0-ef32-4fe1-b104-d5a058d25ebb/1e2511a2-7248-4cea-afb1-80995e2b8f5b"
-          (reference "R9") (unit 1)
+          (reference "R303") (unit 1)
         )
       )
@@
   (symbol (lib_id "Jumper:Jumper_3_Open") (at 71.12 82.55 0) (unit 1)
     (in_bom yes) (on_board yes) (dnp no) (fields_autoplaced)
-    (property "Reference" "JP1" (at 71.12 76.2 0)
+    (property "Reference" "JP301" (at 71.12 76.2 0)
       (effects (font (size 1.27 1.27)))
     )
@@
       (effects (font (size 1.27 1.27)))
     )
-    (property "Footprint" "" (at 71.12 82.55 0)
+    (property "Footprint" "Connector_PinHeader_2.54mm:PinHeader_1x03_P2.54mm_Vertical" (at 71.12 82.55 0)
       (effects (font (size 1.27 1.27)) hide)
     )
@@
       (project "M304B"
         (path "/922fb1f0-ef32-4fe1-b104-d5a058d25ebb/1e2511a2-7248-4cea-afb1-80995e2b8f5b"
-          (reference "JP1") (unit 1)
+          (reference "JP301") (unit 1)
         )
       )
@@
   (symbol (lib_id "power:GND") (at 133.35 101.6 0) (unit 1)
     (in_bom yes) (on_board yes) (dnp no)
-    (property "Reference" "#PWR0161" (at 133.35 107.95 0)
+    (property "Reference" "#PWR0301" (at 133.35 107.95 0)
       (effects (font (size 1.27 1.27)) hide)
     )
@@
       (project "M304B"
         (path "/922fb1f0-ef32-4fe1-b104-d5a058d25ebb/1e2511a2-7248-4cea-afb1-80995e2b8f5b"
-          (reference "#PWR0161") (unit 1)
+          (reference "#PWR0301") (unit 1)
         )
       )
@@
   (symbol (lib_id "Connector_Generic:Conn_01x01") (at 118.11 49.53 270) (mirror x) (unit 1)
     (in_bom yes) (on_board yes) (dnp no)
-    (property "Reference" "SQW1" (at 118.11 45.72 90)
+    (property "Reference" "SQW301" (at 118.11 45.72 90)
       (effects (font (size 1.27 1.27)))
     )
@@
       (project "M304B"
         (path "/922fb1f0-ef32-4fe1-b104-d5a058d25ebb/1e2511a2-7248-4cea-afb1-80995e2b8f5b"
-          (reference "SQW1") (unit 1)
+          (reference "SQW301") (unit 1)
         )
       )
@@
   (symbol (lib_id "Device:R_US") (at 160.02 67.31 0) (unit 1)
     (in_bom yes) (on_board yes) (dnp no) (fields_autoplaced)
-    (property "Reference" "R8" (at 161.671 66.0979 0)
+    (property "Reference" "R305" (at 161.671 66.0979 0)
       (effects (font (size 1.27 1.27)) (justify left))
     )
@@
       (effects (font (size 1.27 1.27)) (justify left))
     )
-    (property "Footprint" "" (at 161.036 67.564 90)
+    (property "Footprint" "Resistor_THT:R_Axial_DIN0207_L6.3mm_D2.5mm_P7.62mm_Horizontal" (at 161.036 67.564 90)
       (effects (font (size 1.27 1.27)) hide)
     )
@@
       (project "M304B"
         (path "/922fb1f0-ef32-4fe1-b104-d5a058d25ebb/1e2511a2-7248-4cea-afb1-80995e2b8f5b"
-          (reference "R8") (unit 1)
+          (reference "R305") (unit 1)
         )
       )
@@
   (symbol (lib_id "Device:R_US") (at 53.34 69.85 0) (unit 1)
     (in_bom yes) (on_board yes) (dnp no) (fields_autoplaced)
-    (property "Reference" "R6" (at 54.991 68.6379 0)
+    (property "Reference" "R301" (at 54.991 68.6379 0)
       (effects (font (size 1.27 1.27)) (justify left))
     )
@@
       (effects (font (size 1.27 1.27)) (justify left))
     )
-    (property "Footprint" "" (at 54.356 70.104 90)
+    (property "Footprint" "Resistor_THT:R_Axial_DIN0207_L6.3mm_D2.5mm_P7.62mm_Horizontal" (at 54.356 70.104 90)
       (effects (font (size 1.27 1.27)) hide)
     )
@@
       (project "M304B"
         (path "/922fb1f0-ef32-4fe1-b104-d5a058d25ebb/1e2511a2-7248-4cea-afb1-80995e2b8f5b"
-          (reference "R6") (unit 1)
+          (reference "R301") (unit 1)
         )
       )
@@
   (symbol (lib_id "Device:Crystal_Small") (at 151.13 92.71 270) (unit 1)
     (in_bom yes) (on_board yes) (dnp no)
-    (property "Reference" "Y1" (at 153.289 91.8753 90)
+    (property "Reference" "Y301" (at 153.289 91.8753 90)
       (effects (font (size 1.27 1.27)) (justify left))
     )
@@
       (project "M304B"
         (path "/922fb1f0-ef32-4fe1-b104-d5a058d25ebb/1e2511a2-7248-4cea-afb1-80995e2b8f5b"
-          (reference "Y1") (unit 1)
+          (reference "Y301") (unit 1)
         )
       )
@@
   (symbol (lib_id "Device:R_US") (at 97.79 91.44 0) (unit 1)
     (in_bom yes) (on_board yes) (dnp no) (fields_autoplaced)
-    (property "Reference" "R5" (at 99.441 90.2279 0)
+    (property "Reference" "R304" (at 99.441 90.2279 0)
       (effects (font (size 1.27 1.27)) (justify left))
     )
@@
       (effects (font (size 1.27 1.27)) (justify left))
     )
-    (property "Footprint" "" (at 98.806 91.694 90)
+    (property "Footprint" "Resistor_THT:R_Axial_DIN0207_L6.3mm_D2.5mm_P7.62mm_Horizontal" (at 98.806 91.694 90)
       (effects (font (size 1.27 1.27)) hide)
     )
@@
       (project "M304B"
         (path "/922fb1f0-ef32-4fe1-b104-d5a058d25ebb/1e2511a2-7248-4cea-afb1-80995e2b8f5b"
-          (reference "R5") (unit 1)
+          (reference "R304") (unit 1)
         )
       )
@@
   (symbol (lib_id "power:GND") (at 166.37 101.6 0) (unit 1)
     (in_bom yes) (on_board yes) (dnp no)
-    (property "Reference" "#PWR0106" (at 166.37 107.95 0)
+    (property "Reference" "#PWR0302" (at 166.37 107.95 0)
       (effects (font (size 1.27 1.27)) hide)
     )
@@
       (project "M304B"
         (path "/922fb1f0-ef32-4fe1-b104-d5a058d25ebb/1e2511a2-7248-4cea-afb1-80995e2b8f5b"
-          (reference "#PWR0106") (unit 1)
+          (reference "#PWR0302") (unit 1)
         )
       )
@@
   (symbol (lib_name "Jumper_3_Open_1") (lib_id "Jumper:Jumper_3_Open") (at 107.95 68.58 0) (unit 1)
     (in_bom yes) (on_board yes) (dnp no) (fields_autoplaced)
-    (property "Reference" "JP2" (at 107.95 62.23 0)
+    (property "Reference" "JP302" (at 107.95 62.23 0)
       (effects (font (size 1.27 1.27)))
     )
@@
       (effects (font (size 1.27 1.27)))
     )
-    (property "Footprint" "" (at 107.95 68.58 0)
+    (property "Footprint" "Connector_PinHeader_2.54mm:PinHeader_1x03_P2.54mm_Vertical" (at 107.95 68.58 0)
       (effects (font (size 1.27 1.27)) hide)
     )
@@
       (project "M304B"
         (path "/922fb1f0-ef32-4fe1-b104-d5a058d25ebb/1e2511a2-7248-4cea-afb1-80995e2b8f5b"
-          (reference "JP2") (unit 1)
+          (reference "JP302") (unit 1)
         )
       )
@@
   (symbol (lib_id "Device:C_Small") (at 152.4 74.93 90) (unit 1)
     (in_bom yes) (on_board yes) (dnp no) (fields_autoplaced)
-    (property "Reference" "C1" (at 152.4063 69.1568 90)
+    (property "Reference" "C301" (at 152.4063 69.1568 90)
       (effects (font (size 1.524 1.524)))
     )
@@
       (project "M304B"
         (path "/922fb1f0-ef32-4fe1-b104-d5a058d25ebb/1e2511a2-7248-4cea-afb1-80995e2b8f5b"
-          (reference "C1") (unit 1)
+          (reference "C301") (unit 1)
         )
       )
@@
   (symbol (lib_id "Device:Battery_Cell") (at 71.12 93.98 0) (unit 1)
     (in_bom yes) (on_board yes) (dnp no)
-    (property "Reference" "BT1" (at 67.31 90.805 0)
+    (property "Reference" "BT301" (at 63.5 90.17 0)
       (effects (font (size 1.27 1.27)) (justify left))
     )
@@
       (project "M304B"
         (path "/922fb1f0-ef32-4fe1-b104-d5a058d25ebb/1e2511a2-7248-4cea-afb1-80995e2b8f5b"
-          (reference "BT1") (unit 1)
+          (reference "BT301") (unit 1)
         )
       )
@@
   (symbol (lib_id "Device:R_US") (at 74.93 60.96 90) (unit 1)
     (in_bom yes) (on_board yes) (dnp no) (fields_autoplaced)
-    (property "Reference" "R4" (at 74.93 55.9267 90)
+    (property "Reference" "R302" (at 74.93 55.9267 90)
       (effects (font (size 1.27 1.27)))
     )
@@
       (effects (font (size 1.27 1.27)))
     )
-    (property "Footprint" "" (at 75.184 59.944 90)
+    (property "Footprint" "Resistor_THT:R_Axial_DIN0207_L6.3mm_D2.5mm_P7.62mm_Horizontal" (at 75.184 59.944 90)
       (effects (font (size 1.27 1.27)) hide)
     )
@@
       (project "M304B"
         (path "/922fb1f0-ef32-4fe1-b104-d5a058d25ebb/1e2511a2-7248-4cea-afb1-80995e2b8f5b"
-          (reference "R4") (unit 1)
+          (reference "R302") (unit 1)
         )
       )
@@
   (symbol (lib_id "Timer_RTC:DS1307+") (at 133.35 88.9 0) (mirror y) (unit 1)
     (in_bom yes) (on_board yes) (dnp no)
-    (property "Reference" "U1" (at 121.92 77.47 0)
+    (property "Reference" "U301" (at 121.92 77.47 0)
       (effects (font (size 1.27 1.27)))
     )
@@
       (project "M304B"
         (path "/922fb1f0-ef32-4fe1-b104-d5a058d25ebb/1e2511a2-7248-4cea-afb1-80995e2b8f5b"
-          (reference "U1") (unit 1)
+          (reference "U301") (unit 1)
         )
       )
@@
   (symbol (lib_id "Diode:1N4148") (at 64.77 67.31 90) (unit 1)
     (in_bom yes) (on_board yes) (dnp no) (fields_autoplaced)
-    (property "Reference" "D1" (at 66.802 66.0979 90)
+    (property "Reference" "D301" (at 66.802 66.0979 90)
       (effects (font (size 1.27 1.27)) (justify right))
     )
@@
       (project "M304B"
         (path "/922fb1f0-ef32-4fe1-b104-d5a058d25ebb/1e2511a2-7248-4cea-afb1-80995e2b8f5b"
-          (reference "D1") (unit 1)
-        )
-      )
+          (reference "D301") (unit 1)
+        )
+      )
